File: KiCad/Ethernet/ethernet.kicad_sch (KiCad schematic)
At the start: 31 parts, among them IC1 74LS32, IC2 74LS688, IC3 74LVC245, IC4 74LVC245, IC5 74LVC245, J1 NKC-Bus, J2 Jumper, J3 Conn_01x09, J5 SBHE_Jumper, J6 A0_Jumper, Q1 BC547, Q2 BC547, SW1 SW_DIP_x04, U1 LT1086-3.3

Commit message: Added layout
Parts:
- Q1, Q2: footprint Package_TO_SOT_THT:TO-92_Inline -> Package_TO_SOT_THT:TO-92_Inline_Wide
Connections:
- net +3V3: now also C5.1
- net VCC: no longer C5.1
- net at IC2.18 (R7), RN1.2 (R1): now also SW1.4; no longer SW1.1
- net at IC2.16 (R6), RN1.3 (R2): now also SW1.3; no longer SW1.2
- net at IC2.14 (R5), RN1.4 (R3): now also SW1.2; no longer SW1.3
- net at IC2.12 (R4), RN1.5 (R4): now also SW1.1; no longer SW1.4
Other:
- moved on the sheet: SW1

Commit message: update to V2.0
Parts:
- removed Q1: BC547, Package_TO_SOT_THT:TO-92_Inline_Wide, symbol Transistor_BJT:BC547
- added C12: 10uF, Capacitor_THT:CP_Radial_D5.0mm_P2.50mm, symbol Device:C_Polarized
- added Q2: BC557, Package_TO_SOT_THT:TO-92_Inline_Wide, symbol Transistor_BJT:BC557
- R2: value 1k -> 220
- renumbered Q2 to Q1
Connections:
- net +3V3: now also C12.1, Q2.3 (E)
- net GND: now also IC3.19 (CE), IC4.19 (CE), IC5.9 (A7), C12.2
- net VCC: no longer R2.2
- net /RD: no longer IC3.1 (A->B), IC4.1 (A->B)
- net /RESET: now also IC5.8 (A6); no longer R1.1
- net at IC5.14 (B4), U2.13b (/IOR): now also IC3.1 (A->B), IC4.1 (A->B)
- net at U2.16b (RESET): now also R2.1; no longer IC5.12 (B6)
- net at IC1.1, IC1.5, IC2.19 (P=R): no longer IC3.19 (CE), IC4.19 (CE)
- net at R1.2: now also Q2.2 (B)
- new net: IC5.12 (B6), R1.1
- new net: Q2.1 (C), R2.2
