File: KiCad/Ethernet/ethernet.kicad_pcb (KiCad board)
At the start: 2 copper layers, 100 x 100 mm, 31 parts, among them IC1 74LS32, IC2 74LS688, IC3 74LVC245, IC4 74LVC245, IC5 74LVC245, J1 NKC-Bus, J2 Jumper, J3 Ext, J5 SBHE_Jumper, J6 A0_Jumper, Q1 BC547, Q2 BC547, SW1 SW_DIP_x04, U1 LT1086-3.3

Commit message: update to V2.0
Parts:
- removed the Q1 at (127.0, 163.8)
- added C12: 10uF, Capacitor_THT:CP_Radial_D5.0mm_P2.50mm, F.Cu at (114.9, 88.9)
- added Q2: BC557, Package_TO_SOT_THT:TO-92_Inline_Wide, F.Cu at (122.2, 158.2)
- J3: value Ext -> Conn_01x09
- R2: value 1k -> 220
- moved R3 57.8 mm to (130.6, 146.3), turned to 90 degrees
- moved R2 18.8 mm to (126.6, 136.1), turned to -90 degrees
- moved J3 8.89 mm to (71.1, 88.9)
- moved R1 5.93 mm to (126.7, 150.6), turned to -90 degrees
- moved C5 5.12 mm to (123.2, 89.0)
- moved U2 5.08 mm to (128.3, 95.2)
- moved J5 3.01 mm to (90.3, 88.9), turned to 90 degrees
- moved Q1 2.03 mm to (131.4, 163.1)
- renumbered Q2 to Q1
Connections:
- IC3 pad 1: //RD -> Net-(IC3-A->B)
- IC3 pad 19: Net-(IC2-P=R) -> GND
- IC4 pad 1: //RD -> Net-(IC3-A->B)
- IC4 pad 19: Net-(IC2-P=R) -> GND
- IC5 pad 14: Net-(IC5-B4) -> Net-(IC3-A->B)
- IC5 pad 8: Net-(IC5-A6) -> //RESET
- IC5 pad 9: Net-(IC5-A6) -> GND
- R1 pad 1: //RESET -> Net-(IC5-B6)
- R2 pad 1: Net-(IC5-A6) -> Net-(U2-RESET)
- R2 pad 2: VCC -> Net-(Q2-C)
- U2 pad 13b: Net-(IC5-B4) -> Net-(IC3-A->B)
- U2 pad 16b: Net-(IC5-B6) -> Net-(U2-RESET)
Routing:
- net Net-(IC3-A->B): track 0.00 -> 140.3 mm, vias 0 -> 3
- net //RD: track 144.3 -> 56.9 mm, vias 7 -> 2
- net Net-(Q1-B): track 87.0 -> 15.4 mm, vias 2 -> 0
- net Net-(IC5-B6): track 74.2 -> 17.6 mm
- net Net-(IC5-B4): track 56.6 -> 0.00 mm
- net Net-(IC2-P=R): track 103.0 -> 48.7 mm, vias 3 -> 1
- net Net-(U2-IRQ0): track 12.2 -> 47.5 mm, vias 0 -> 2
- net Net-(IC5-B0): track 114.6 -> 80.5 mm, vias 5 -> 3
- net Net-(IC5-A6): track 34.0 -> 0.00 mm, vias 2 -> 0
- net Net-(IC5-B5): track 64.4 -> 42.4 mm
- net Net-(IC3-B0): track 49.5 -> 31.0 mm, vias 0 -> 2
- net Net-(IC3-B1): track 52.8 -> 35.0 mm, vias 0 -> 3
- net Net-(Q2-B): track 21.1 -> 4.57 mm
- net Net-(IC5-A5): track 67.5 -> 51.2 mm
- net Net-(U2-RESET): track 0.00 -> 16.3 mm, vias 0 -> 1
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
Commit message: update
Routing:
- net //RD: track 56.9 -> 55.2 mm
- net /A3: track 27.8 -> 26.8 mm
- net Net-(IC5-B6): track 17.6 -> 16.6 mm
- net /D7: track 21.1 -> 20.1 mm
- net Net-(IC3-B1): track 35.0 -> 34.0 mm
- net Net-(J5-Pin_2): track 59.5 -> 58.7 mm
- net Net-(IC2-P=R): track 48.7 -> 48.0 mm
- net Net-(IC5-B3): track 44.5 -> 43.8 mm
- net Net-(IC3-A->B): track 140.3 -> 139.6 mm
- net /D12: track 31.9 -> 31.2 mm
- net /D13: track 33.8 -> 33.2 mm
- net /D14: track 38.4 -> 37.9 mm
- net //RESET: track 19.8 -> 19.2 mm

Commit message: minor bugfix
Routing:
- net +3V3: track 20.1 -> 21.0 mm
Changed lines of the file:
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@@
   (segment (start 90.17 124.714) (end 90.678 125.222) (width 0.25) (layer "B.Cu") (net 2))
   (segment (start 90.17 120.65) (end 90.17 124.714) (width 0.25) (layer "B.Cu") (net 2))
-  (segment (start 49.53 122.26) (end 49.53 124.42) (width 0.25) (layer "F.Cu") (net 3))
-  (segment (start 56.642 120.015) (end 57.19 120.015) (width 0.25) (layer "F.Cu") (net 3))
-  (segment (start 55.753 120.015) (end 56.642 120.015) (width 0.25) (layer "F.Cu") (net 3))
-  (segment (start 49.657 120.015) (end 55.753 120.015) (width 0.25) (layer "F.Cu") (net 3))
-  (segment (start 49.53 122.26) (end 49.53 119.888) (width 0.25) (layer "F.Cu") (net 3))
-  (segment (start 57.19 120.015) (end 59.055 121.88) (width 0.25) (layer "F.Cu") (net 3))
-  (segment (start 49.53 124.42) (end 45.68 128.27) (width 0.25) (layer "F.Cu") (net 3))
+  (segment (start 49.53 122.26) (end 49.53 124.42) (width 1) (layer "F.Cu") (net 3))
+  (segment (start 56.642 120.015) (end 56.7436 120.015) (width 1) (layer "F.Cu") (net 3))
+  (segment (start 49.53 122.26) (end 49.53 119.0752) (width 1) (layer "F.Cu") (net 3))
+  (segment (start 55.753 120.015) (end 56.1086 120.015) (width 1) (layer "F.Cu") (net 3))
+  (segment (start 56.1086 120.015) (end 56.642 120.015) (width 1) (layer "F.Cu") (net 3))
+  (segment (start 49.657 120.015) (end 55.753 120.015) (width 1) (layer "F.Cu") (net 3))
+  (segment (start 57.19 120.015) (end 59.055 121.88) (width 1) (layer "F.Cu") (net 3))
+  (segment (start 56.7436 120.015) (end 57.19 120.015) (width 1) (layer "F.Cu") (net 3))
+  (segment (start 49.53 124.42) (end 45.68 128.27) (width 1) (layer "F.Cu") (net 3))
   (via (at 45.212 109.982) (size 0.6) (drill 0.4) (layers "F.Cu" "B.Cu") (free) (net 3))
   (via (at 45.212 107.95) (size 0.6) (drill 0.4) (layers "F.Cu" "B.Cu") (free) (net 3))
@@
   (via (at 53.848 112.014) (size 0.6) (drill 0.4) (layers "F.Cu" "B.Cu") (free) (net 3))
   (via (at 53.848 105.664) (size 0.6) (drill 0.4) (layers "F.Cu" "B.Cu") (free) (net 3))
-  (via (at 56.642 120.015) (size 0.6) (drill 0.4) (layers "F.Cu" "B.Cu") (net 3))
   (via (at 49.53 113.919) (size 0.6) (drill 0.4) (layers "F.Cu" "B.Cu") (free) (net 3))
   (via (at 45.212 112.014) (size 0.6) (drill 0.4) (layers "F.Cu" "B.Cu") (free) (net 3))
   (via (at 53.848 103.505) (size 0.6) (drill 0.4) (layers "F.Cu" "B.Cu") (free) (net 3))
   (via (at 49.53 110.109) (size 0.6) (drill 0.4) (layers "F.Cu" "B.Cu") (free) (net 3))
+  (via (at 56.7436 120.015) (size 0.6) (drill 0.3) (layers "F.Cu" "B.Cu") (net 3))
   (via (at 53.848 113.919) (size 0.6) (drill 0.4) (layers "F.Cu" "B.Cu") (free) (net 3))
   (via (at 53.848 107.823) (size 0.6) (drill 0.4) (layers "F.Cu" "B.Cu") (free) (net 3))
@@
   (via (at 53.848 110.109) (size 0.6) (drill 0.4) (layers "F.Cu" "B.Cu") (free) (net 3))
   (via (at 45.212 103.505) (size 0.6) (drill 0.4) (layers "F.Cu" "B.Cu") (free) (net 3))
+  (via (at 56.1086 120.015) (size 0.6) (drill 0.3) (layers "F.Cu" "B.Cu") (net 3))
   (via (at 45.212 105.537) (size 0.6) (drill 0.4) (layers "F.Cu" "B.Cu") (free) (net 3))
-  (via (at 55.753 120.015) (size 0.6) (drill 0.4) (layers "F.Cu" "B.Cu") (net 3))
   (segment (start 99.380411 137.703189) (end 96.266 140.8176) (width 0.25) (layer "F.Cu") (net 4))
   (segment (start 96.266 147.32) (end 98.176 149.23) (width 0.25) (layer "F.Cu") (net 4))
